File: Hardware/$stm32f103-ibus.sch (KiCad schematic (older format))
At the start: 14 parts

Commit message: 1.Supports BMW E38 thermostat heater control according to information from I-Bus 2.Modify circuit 3.Add data sheet
Connections:
- wire segments 37 -> 38
Changed lines of the file:
@@
 Wire Wire Line
 	2700 1300 2850 1300
+$Comp
+L +5V #PWR?
+U 1 1 598D88F3
+P 4250 4600
+F 0 "#PWR?" H 4250 4690 20  0001 C CNN
+F 1 "+5V" H 4250 4690 30  0000 C CNN
+F 2 "" H 4250 4600 60  0000 C CNN
+F 3 "" H 4250 4600 60  0000 C CNN
+	1    4250 4600
+	1    0    0    -1
+$EndComp
+Wire Wire Line
+	4400 4600 4250 4600
 $EndSCHEMATC
